Commit message: changed made

File: mycobot_280jn_sim/urdf/mycobot_280jn_sim.urdf.xacro (robot description, xacro)
@@ -220,9 +220,9 @@
     <material name="mycobot_dark_gray"/>
     </visual>
-    <collision>
-      <geometry>
-       <mesh filename="package://mycobot_description/urdf/adaptive_gripper/gripper_base.dae"/>
-      </geometry>
-    <origin xyz = "0.0 0 -0.012 " rpy = " 0 0 0"/>
+    <collision name="gripper_base_collision">
+      <origin xyz="0 0 -0.012" rpy="0 0 0"/>
+      <geometry>
+        <box size="0.08 0.06 0.04"/>
+      </geometry>
     </collision>
   </link>

Commit message: something wrong

File: mycobot_280jn_sim/urdf/mycobot_280jn_sim.urdf.xacro (robot description, xacro)
@@ -237,8 +237,8 @@
     </visual>
     <collision>
-      <geometry>
-       <mesh filename="package://mycobot_description/urdf/adaptive_gripper/gripper_left1.dae"/>
-      </geometry>
-        <origin xyz = "0.039 -0.0133 -0.012 " rpy = " 0 0 0"/>
+      <origin xyz="0.039 -0.0133 -0.012" rpy="0 0 0"/>
+      <geometry>
+        <box size="0.04 0.018 0.022"/>
+      </geometry>
     </collision>
   </link>
@@ -253,8 +253,8 @@
     </visual>
     <collision>
-      <geometry>
-       <mesh filename="package://mycobot_description/urdf/adaptive_gripper/gripper_left2.dae"/>
-      </geometry>
-        <origin xyz = "0.005 -0.0195 -0.012 " rpy = " 0 0 0"/>
+      <origin xyz="0.005 -0.0195 -0.012" rpy="0 0 0"/>
+      <geometry>
+        <box size="0.04 0.018 0.022"/>
+      </geometry>
     </collision>
   </link>
@@ -269,8 +269,8 @@
     </visual>
     <collision>
-      <geometry>
-       <mesh filename="package://mycobot_description/urdf/adaptive_gripper/gripper_left3.dae"/>
-      </geometry>
-    <origin xyz = "0.012 0.0025 -0.012 " rpy = " 0 0 0"/>
+      <origin xyz="0.012 0.0025 -0.012" rpy="0 0 0"/>
+      <geometry>
+        <box size="0.03 0.012 0.018"/>
+      </geometry>
     </collision>
   </link>
@@ -285,8 +285,8 @@
     </visual>
     <collision>
-      <geometry>
-       <mesh filename="package://mycobot_description/urdf/adaptive_gripper/gripper_right1.dae"/>
-      </geometry>
-        <origin xyz = "-0.039 -0.0133 -0.012 " rpy = " 0 0 0"/>
+      <origin xyz="-0.039 -0.0133 -0.012" rpy="0 0 0"/>
+      <geometry>
+        <box size="0.04 0.018 0.022"/>
+      </geometry>
     </collision>
   </link>
@@ -301,8 +301,8 @@
     </visual>
     <collision>
-      <geometry>
-       <mesh filename="package://mycobot_description/urdf/adaptive_gripper/gripper_right2.dae"/>
-      </geometry>
-        <origin xyz = "-0.005 -0.0195 -0.012 " rpy = " 0 0 0"/>
+      <origin xyz="-0.005 -0.0195 -0.012" rpy="0 0 0"/>
+      <geometry>
+        <box size="0.04 0.018 0.022"/>
+      </geometry>
     </collision>
   </link>
@@ -317,8 +317,8 @@
     </visual>
     <collision>
-      <geometry>
-       <mesh filename="package://mycobot_description/urdf/adaptive_gripper/gripper_right3.dae"/>
-      </geometry>
-    <origin xyz = "-0.012 0.0025 -0.012" rpy = " 0 0 0"/>
+      <origin xyz="-0.012 0.0025 -0.012" rpy="0 0 0"/>
+      <geometry>
+        <box size="0.03 0.012 0.018"/>
+      </geometry>
     </collision>
   </link>
@@ -536,4 +536,47 @@
     </joint>
   </ros2_control>
+  <!-- Match pick_cube friction so finger–cube contacts grip reliably. -->
+  <gazebo reference="gripper_base">
+    <mu1>2.5</mu1>
+    <mu2>2.5</mu2>
+    <kp>75000</kp>
+    <kd>10</kd>
+  </gazebo>
+  <gazebo reference="gripper_left1">
+    <mu1>2.5</mu1>
+    <mu2>2.5</mu2>
+    <kp>75000</kp>
+    <kd>10</kd>
+  </gazebo>
+  <gazebo reference="gripper_left2">
+    <mu1>2.5</mu1>
+    <mu2>2.5</mu2>
+    <kp>75000</kp>
+    <kd>10</kd>
+  </gazebo>
+  <gazebo reference="gripper_left3">
+    <mu1>2.5</mu1>
+    <mu2>2.5</mu2>
+    <kp>75000</kp>
+    <kd>10</kd>
+  </gazebo>
+  <gazebo reference="gripper_right1">
+    <mu1>2.5</mu1>
+    <mu2>2.5</mu2>
+    <kp>75000</kp>
+    <kd>10</kd>
+  </gazebo>
+  <gazebo reference="gripper_right2">
+    <mu1>2.5</mu1>
+    <mu2>2.5</mu2>
+    <kp>75000</kp>
+    <kd>10</kd>
+  </gazebo>
+  <gazebo reference="gripper_right3">
+    <mu1>2.5</mu1>
+    <mu2>2.5</mu2>
+    <kp>75000</kp>
+    <kd>10</kd>
+  </gazebo>
   <!-- This Gazebo system creates controller_manager and reads the YAML. -->
   <gazebo>
@@ -544,4 +587,6 @@
       <parameters>$(find mycobot_280jn_sim)/config/controllers.yaml</parameters>
       <controller_manager_name>controller_manager</controller_manager_name>
+      <!-- Softer joint tracking reduces penetration through table/cube. -->
+      <position_proportional_gain>0.25</position_proportional_gain>
     </plugin>
   </gazebo>

Commit message: fixes

File: mycobot_280jn_sim/urdf/mycobot_280jn_sim.urdf.xacro (robot description, xacro)
@@ -239,5 +239,5 @@
       <origin xyz="0.039 -0.0133 -0.012" rpy="0 0 0"/>
       <geometry>
-        <box size="0.04 0.018 0.022"/>
+        <mesh filename="package://mycobot_description/urdf/adaptive_gripper/gripper_left1.dae"/>
       </geometry>
     </collision>
@@ -255,5 +255,5 @@
       <origin xyz="0.005 -0.0195 -0.012" rpy="0 0 0"/>
       <geometry>
-        <box size="0.04 0.018 0.022"/>
+        <mesh filename="package://mycobot_description/urdf/adaptive_gripper/gripper_left2.dae"/>
       </geometry>
     </collision>
@@ -271,5 +271,5 @@
       <origin xyz="0.012 0.0025 -0.012" rpy="0 0 0"/>
       <geometry>
-        <box size="0.03 0.012 0.018"/>
+        <mesh filename="package://mycobot_description/urdf/adaptive_gripper/gripper_left3.dae"/>
       </geometry>
     </collision>
@@ -287,5 +287,5 @@
       <origin xyz="-0.039 -0.0133 -0.012" rpy="0 0 0"/>
       <geometry>
-        <box size="0.04 0.018 0.022"/>
+        <mesh filename="package://mycobot_description/urdf/adaptive_gripper/gripper_right1.dae"/>
       </geometry>
     </collision>
@@ -303,5 +303,5 @@
       <origin xyz="-0.005 -0.0195 -0.012" rpy="0 0 0"/>
       <geometry>
-        <box size="0.04 0.018 0.022"/>
+        <mesh filename="package://mycobot_description/urdf/adaptive_gripper/gripper_right2.dae"/>
       </geometry>
     </collision>
@@ -319,5 +319,5 @@
       <origin xyz="-0.012 0.0025 -0.012" rpy="0 0 0"/>
       <geometry>
-        <box size="0.03 0.012 0.018"/>
+        <mesh filename="package://mycobot_description/urdf/adaptive_gripper/gripper_right3.dae"/>
       </geometry>
     </collision>
@@ -587,6 +587,5 @@
       <parameters>$(find mycobot_280jn_sim)/config/controllers.yaml</parameters>
       <controller_manager_name>controller_manager</controller_manager_name>
-      <!-- Softer joint tracking reduces penetration through table/cube. -->
-      <position_proportional_gain>0.25</position_proportional_gain>
+      <position_proportional_gain>1.0</position_proportional_gain>
     </plugin>
   </gazebo>
