Commit message: Fix Jazzy ros2_control mimic joints and document launch errors.
Remove command interfaces from URDF mimic followers; Jazzy parses
URDF mimic tags instead of deprecated ros2_control mimic params.

Co-authored-by: Cursor <cursoragent@cursor.com>

File: mycobot_280jn_sim/urdf/mycobot_280jn_sim.urdf.xacro (robot description, xacro)
@@ -488,10 +488,7 @@
       <state_interface name="velocity"/>
     </joint>
-    <!-- Followers are driven by gz_ros2_control mimic params (not Gazebo's
-         URDF <mimic> joints, which create conflicting *_mimic joints). -->
+    <!-- Jazzy: mimic followers use URDF <mimic> tags; state interfaces only
+         (command interfaces on mimic joints are rejected by ros2_control). -->
     <joint name="gripper_base_to_gripper_left2">
-      <param name="mimic">gripper_controller</param>
-      <param name="multiplier">1.0</param>
-      <command_interface name="position"/>
       <state_interface name="position">
         <param name="initial_value">0.0</param>
@@ -500,7 +497,4 @@
     </joint>
     <joint name="gripper_left3_to_gripper_left1">
-      <param name="mimic">gripper_controller</param>
-      <param name="multiplier">-1.0</param>
-      <command_interface name="position"/>
       <state_interface name="position">
         <param name="initial_value">0.0</param>
@@ -509,7 +503,4 @@
     </joint>
     <joint name="gripper_base_to_gripper_right3">
-      <param name="mimic">gripper_controller</param>
-      <param name="multiplier">-1.0</param>
-      <command_interface name="position"/>
       <state_interface name="position">
         <param name="initial_value">0.0</param>
@@ -518,7 +509,4 @@
     </joint>
     <joint name="gripper_base_to_gripper_right2">
-      <param name="mimic">gripper_controller</param>
-      <param name="multiplier">-1.0</param>
-      <command_interface name="position"/>
       <state_interface name="position">
         <param name="initial_value">0.0</param>
@@ -527,7 +515,4 @@
     </joint>
     <joint name="gripper_right3_to_gripper_right1">
-      <param name="mimic">gripper_controller</param>
-      <param name="multiplier">1.0</param>
-      <command_interface name="position"/>
       <state_interface name="position">
         <param name="initial_value">0.0</param>
